File: hardware/display/display.kicad_sch (KiCad schematic)
At the start: 425 parts, among them J1 Power Connector, J2 Data Connector

Commit message: Updated Mounting Holes
M2 screw holes for M2x4mm screws into top of case.
Parts:
- H1, H2, H3, H4: footprint MountingHole:MountingHole_3.2mm_M3_DIN965_Pad -> MountingHole:MountingHole_2.2mm_M2_Pad
Changed lines of the file:
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@@
 			)
 		)
-		(property "Footprint" "MountingHole:MountingHole_3.2mm_M3_DIN965_Pad"
+		(property "Footprint" "MountingHole:MountingHole_2.2mm_M2_Pad"
 			(at 287.02 228.6 0)
 			(effects
@@
 			)
 		)
-		(property "Footprint" "MountingHole:MountingHole_3.2mm_M3_DIN965_Pad"
+		(property "Footprint" "MountingHole:MountingHole_2.2mm_M2_Pad"
 			(at 307.34 228.6 0)
 			(effects
@@
 			)
 		)
-		(property "Footprint" "MountingHole:MountingHole_3.2mm_M3_DIN965_Pad"
+		(property "Footprint" "MountingHole:MountingHole_2.2mm_M2_Pad"
 			(at 287.02 222.25 0)
 			(effects
@@
 			)
 		)
-		(property "Footprint" "MountingHole:MountingHole_3.2mm_M3_DIN965_Pad"
+		(property "Footprint" "MountingHole:MountingHole_2.2mm_M2_Pad"
 			(at 307.34 222.25 0)
 			(effects

Commit message: Updated Mounting Holes
Made display holes M3

Matching hole pattern on motherboard to mount display.

Distributed 4, M3 mounting holes throuhout motherboard
Parts:
- H1, H2, H3, H4: footprint MountingHole:MountingHole_2.2mm_M2_Pad -> MountingHole:MountingHole_3.2mm_M3_Pad
Changed lines of the file:
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@@
 			)
 		)
-		(property "Footprint" "MountingHole:MountingHole_2.2mm_M2_Pad"
+		(property "Footprint" "MountingHole:MountingHole_3.2mm_M3_Pad"
 			(at 287.02 228.6 0)
 			(effects
@@
 			)
 		)
-		(property "Footprint" "MountingHole:MountingHole_2.2mm_M2_Pad"
+		(property "Footprint" "MountingHole:MountingHole_3.2mm_M3_Pad"
 			(at 307.34 228.6 0)
 			(effects
@@
 			)
 		)
-		(property "Footprint" "MountingHole:MountingHole_2.2mm_M2_Pad"
+		(property "Footprint" "MountingHole:MountingHole_3.2mm_M3_Pad"
 			(at 287.02 222.25 0)
 			(effects
@@
 			)
 		)
-		(property "Footprint" "MountingHole:MountingHole_2.2mm_M2_Pad"
+		(property "Footprint" "MountingHole:MountingHole_3.2mm_M3_Pad"
 			(at 307.34 222.25 0)
 			(effects

Commit message: WIP Continued – Display
Parts:
- removed C41, C42, C43, C44, C45, C46, C47, C48, C49, C50: 0.1uF, Capacitor_SMD:C_0402_1005Metric_Pad0.74x0.62mm_HandSolder, symbol Device:C_Small
- added C71, C72, C73, C74, C75, C76, C77, C78, C79, C80: 0.1uF, Capacitor_SMD:C_0402_1005Metric_Pad0.74x0.62mm_HandSolder, symbol Device:C_Small
- renumbered C71 to C41, C72 to C42, C73 to C43, C74 to C44, C76 to C45, C78 to C46, C75 to C47, C77 to C48, C79 to C49, C80 to C50
Connections:
- net GND: now also C71.2, C72.2, C73.2, C74.2, C75.2, C76.2, C77.2, C78.2, C79.2, C80.2
- net VDD: now also C1.1, C10.1, C11.1, C12.1, C13.1, C14.1, C15.1, C16.1, C17.1, C18.1, C19.1, C2.1, C20.1, C21.1, C22.1, C23.1, C24.1, C25.1, C26.1, C27.1, C28.1, C29.1, C3.1, C30.1, C31.1, C32.1, C33.1, C34.1, C35.1, C36.1, C37.1, C38.1, C39.1, C4.1, C40.1, C41.1, C42.1, C43.1, C44.1, C45.1, C46.1, C47.1, C48.1, C49.1, C5.1, C50.1, C51.1, C52.1, C53.1, C54.1, C55.1, C56.1, C57.1, C58.1, C59.1, C6.1, C60.1, C61.1, C62.1, C63.1, C64.1, C65.1, C66.1, C67.1, C68.1, C69.1, C7.1, C70.1, C8.1, C9.1, C71.1, C72.1, C73.1, C74.1, C75.1, C76.1, C77.1, C78.1, C79.1, C80.1
- net at D300.1 (DOUT), D301.3 (DIN): no longer C45.1
- net at D216.1 (DOUT), D217.3 (DIN): no longer C55.1
- net at D16.1 (DOUT), D17.3 (DIN): no longer C5.1
- net at D76.1 (DOUT), D77.3 (DIN): no longer C20.1
- net at D316.1 (DOUT), D317.3 (DIN): no longer C50.1
- net at D121.3 (DIN), R4.2: no longer C31.1
- net at D64.1 (DOUT), D65.3 (DIN): no longer C17.1
- net at D4.1 (DOUT), D5.3 (DIN): no longer C2.1
- net at D281.3 (DIN), R8.2: no longer C41.1
- net at D104.1 (DOUT), D105.3 (DIN): no longer C27.1
- net at D224.1 (DOUT), D225.3 (DIN): no longer C57.1
- net at D124.1 (DOUT), D125.3 (DIN): no longer C32.1
- net at D60.1 (DOUT), D61.3 (DIN): no longer C16.1
- net at D264.1 (DOUT), D265.3 (DIN): no longer C67.1
- net at D68.1 (DOUT), D69.3 (DIN): no longer C18.1
- net at D241.3 (DIN), R7.2: no longer C61.1
- net at D112.1 (DOUT), D113.3 (DIN): no longer C29.1
- net at D308.1 (DOUT), D309.3 (DIN): no longer C46.1
- net at D312.1 (DOUT), D313.3 (DIN): no longer C49.1
- net at D8.1 (DOUT), D9.3 (DIN): no longer C3.1
- net at D41.3 (DIN), R2.2: no longer C11.1
- net at D20.1 (DOUT), D21.3 (DIN): no longer C6.1
- net at D260.1 (DOUT), D261.3 (DIN): no longer C66.1
- net at D276.1 (DOUT), D277.3 (DIN): no longer C70.1
- net at D256.1 (DOUT), D257.3 (DIN): no longer C65.1
- net at D248.1 (DOUT), D249.3 (DIN): no longer C63.1
- net at D136.1 (DOUT), D137.3 (DIN): no longer C35.1
- net at D96.1 (DOUT), D97.3 (DIN): no longer C25.1
- net at D32.1 (DOUT), D33.3 (DIN): no longer C9.1
- net at D201.3 (DIN), R6.2: no longer C51.1
- net at D156.1 (DOUT), D157.3 (DIN): no longer C40.1
- net at D236.1 (DOUT), D237.3 (DIN): no longer C60.1
- net at D116.1 (DOUT), D117.3 (DIN): no longer C30.1
- net at D232.1 (DOUT), D233.3 (DIN): no longer C59.1
- net at D292.1 (DOUT), D293.3 (DIN): no longer C44.1
- net at D204.1 (DOUT), D205.3 (DIN): no longer C52.1
- net at D284.1 (DOUT), D285.3 (DIN): no longer C42.1
- net at D72.1 (DOUT), D73.3 (DIN): no longer C19.1
- net at D81.3 (DIN), R3.2: no longer C21.1
- net at D108.1 (DOUT), D109.3 (DIN): no longer C28.1
- net at D48.1 (DOUT), D49.3 (DIN): no longer C13.1
- net at D1.3 (DIN), R1.2: no longer C1.1
- net at D140.1 (DOUT), D141.3 (DIN): no longer C36.1
- net at D296.1 (DOUT), D297.3 (DIN): no longer C47.1
- net at D252.1 (DOUT), D253.3 (DIN): no longer C64.1
- net at D212.1 (DOUT), D213.3 (DIN): no longer C54.1
- net at D208.1 (DOUT), D209.3 (DIN): no longer C53.1
- net at D228.1 (DOUT), D229.3 (DIN): no longer C58.1
- net at D24.1 (DOUT), D25.3 (DIN): no longer C7.1
- net at D128.1 (DOUT), D129.3 (DIN): no longer C33.1
- net at D100.1 (DOUT), D101.3 (DIN): no longer C26.1
- net at D52.1 (DOUT), D53.3 (DIN): no longer C14.1
- net at D288.1 (DOUT), D289.3 (DIN): no longer C43.1
- net at D88.1 (DOUT), D89.3 (DIN): no longer C23.1
- net at D272.1 (DOUT), D273.3 (DIN): no longer C69.1
- net at D304.1 (DOUT), D305.3 (DIN): no longer C48.1
- net at D92.1 (DOUT), D93.3 (DIN): no longer C24.1
- net at D144.1 (DOUT), D145.3 (DIN): no longer C37.1
- net at D132.1 (DOUT), D133.3 (DIN): no longer C34.1
- net at D44.1 (DOUT), D45.3 (DIN): no longer C12.1
- net at D56.1 (DOUT), D57.3 (DIN): no longer C15.1
- net at D244.1 (DOUT), D245.3 (DIN): no longer C62.1
- net at D220.1 (DOUT), D221.3 (DIN): no longer C56.1
- net at D28.1 (DOUT), D29.3 (DIN): no longer C8.1
- net at D36.1 (DOUT), D37.3 (DIN): no longer C10.1
- net at D148.1 (DOUT), D149.3 (DIN): no longer C38.1
- net at D84.1 (DOUT), D85.3 (DIN): no longer C22.1
- net at D268.1 (DOUT), D269.3 (DIN): no longer C68.1
- net at D12.1 (DOUT), D13.3 (DIN): no longer C4.1
- net at D152.1 (DOUT), D153.3 (DIN): no longer C39.1
Other:
- moved on the sheet: C41, C42, C43, C44, C45, C46, C47, C48, C49, C50
